Commit message: [add] robotis model add ft sensor

File: AAAAA/robotis_op_description/robots/robotis_op.urdf (robot description, URDF)
Before this commit: robot robotis_op2, 31 links, 30 joints
Links:
- link MP_ARM_GRIPPER_FIX_DUMMY_L: mass 0.01 -> 0.010
- link MP_ARM_GRIPPER_FIX_DUMMY_R: mass 0.01 -> 0.010
- link MP_ARM_GRIPPER_FIX_L: mass 0.01 -> 0.010
- link MP_ARM_GRIPPER_FIX_R: mass 0.01 -> 0.010
- link MP_ARM_GRIPPER_MOV_L: mass 0.01 -> 0.010
- link MP_ARM_GRIPPER_MOV_R: mass 0.01 -> 0.010
- link MP_ARM_LOW_L: mass 0.01 -> 0.059288504
- link MP_BACK_L: mass 0.01 -> 0.010
- link MP_BACK_R: mass 0.01 -> 0.010
- link MP_PELVIS_L: mass 0.197 -> 0.167
- link MP_THIGH2_L: mass 0.0070309794 -> 0.11904336
- link MP_TIBIA_L: mass 0.0070309794 -> 0.070309794

File: AAAAA/robotis_op_description/urdf/leg/robotis_op_leg.urdf.xacro (robot description, xacro)
@@ -1,228 +1,249 @@
 <?xml version="1.0"?>
+<!-- ROBOTIS-OP2 leg urdf.  Add force-torque sensor for calc ZMP -->
 <!-- Set the robot's name -->
 <robot  name="robotis_op2" xmlns:xacro="http://www.ros.org/wiki/xacro">
   <xacro:macro name="robotis_op_leg_macro">
- <link name="MP_PELVIS_L" >
-    <inertial>
+    <link name="MP_PELVIS_L" >
+      <inertial>
       <origin xyz="0.000000 0.000480 0.018437" />
       <mass value="0.167"/>
       <inertia ixx="0.12259691"  ixy="0.00071127469"  ixz="0.00081143913" iyx="0.00071127469" iyy="0.11066637" iyz="-0.0071635476" izx="0.00081143913" izy="-0.0071635476" izz="0.041877668" />
-    </inertial>
-    <pelvis_l_collision_geom_macro />
-    <pelvis_l_visual_geom_macro />
-  </link>
-  <link name="MP_THIGH1_L" >
-    <inertial>
-      <origin xyz="0.000079 0.018242 0.013873" />
-      <mass value="0.11904336"/>
-      <inertia ixx="0.097950272"  ixy="0.0012119368"  ixz="-0.00021223016" iyx="0.00122119368" iyy="0.032848287" iyz="-0.0019474021" izx="-0.00021223016" izy="-0.0019474021" izz="0.11493509" />
-    </inertial>
-    <thigh1_l_collision_geom_macro />
-    <thigh1_l_visual_geom_macro />
-  </link>
-  <link name="MP_THIGH2_L" >
-    <inertial>
-      <origin xyz="-0.062965 -0.000323 0.000692" />
-      <mass value="0.11904336"/>
-      <inertia ixx="0.097950272"  ixy="0.0012119368"  ixz="-0.00021223016" iyx="0.00122119368" iyy="0.032848287" iyz="-0.0019474021" izx="-0.00021223016" izy="-0.0019474021" izz="0.11493509" />
-    </inertial>
-    <thigh2_l_collision_geom_macro />
-    <thigh2_l_visual_geom_macro />
-  </link>
-  <link name="MP_TIBIA_L" >
-    <inertial>
-      <origin xyz="-0.053955 0.006548 -0.000592" />
-      <mass value="0.070309794"/>
-      <inertia ixx="0.093369608"  ixy="-0.00093567395"  ixz="-0.00023992085" iyx="-0.00093567395" iyy="0.046295534" iyz="-0.012858493" izx="-0.00023992085" izy="-0.012858493" izz="0.11351516" />
-    </inertial>
-    <tibia_l_collision_geom_macro />
-    <tibia_l_visual_geom_macro />
-  </link>
-  <link name="MP_ANKLE1_L" >
-    <inertial>
-      <origin xyz="-0.000214 -0.018536 0.013873" />
-      <mass value="0.16710792"/>
-      <inertia ixx="0.12079175"  ixy="-0.00079781067"  ixz="-0.00039322246" iyx="-0.00079781067" iyy="0.10885465" iyz="0.0070770117" izx="-0.00039322246" izy="0.0070770117" izz="0.041871103" />
-    </inertial>
-    <ankle1_l_collision_geom_macro />
-    <ankle1_l_visual_geom_macro />
-  </link>
-  <link name="MP_ANKLE2_L" >
-    <inertial>
-      <origin xyz="-0.025995 -0.009506 -0.000503" />
-      <mass value="0.0794462"/>
-      <inertia ixx="0.12079175"  ixy="-0.00079781067"  ixz="-0.00039322246" iyx="-0.00079781067" iyy="0.10885465" iyz="0.0070770117" izx="-0.00039322246" izy="0.0070770117" izz="0.041871103" />
-    </inertial>
-    <ankle2_l_collision_geom_macro />
-    <ankle2_l_visual_geom_macro />
-  </link>
-  <link name="MP_PELVIS_R" >
-    <inertial>
-      <origin xyz="0.000000 0.000480 0.018437" />
-      <mass value="0.197"/>
-      <inertia ixx="0.12259691"  ixy="0.00071127469"  ixz="0.00081143913" iyx="0.00071127469" iyy="0.11066637" iyz="-0.0071635476" izx="0.00081143913" izy="-0.0071635476" izz="0.041877668" />
-    </inertial>
-    <pelvis_r_collision_geom_macro />
-    <pelvis_r_visual_geom_macro />
-  </link>
-  <link name="MP_THIGH1_R" >
-    <inertial>
-      <origin xyz="0.000079 -0.018242 0.0138735" />
-      <mass value="0.11904336"/>
-      <inertia ixx="0.097950272"  ixy="0.0012119368"  ixz="-0.00021223016" iyx="0.00122119368" iyy="0.032848287" iyz="-0.0019474021" izx="-0.00021223016" izy="-0.0019474021" izz="0.11493509" />
-    </inertial>
-    <thigh1_r_collision_geom_macro />
-    <thigh1_r_visual_geom_macro />
-  </link>
-  <link name="MP_THIGH2_R" >
-    <inertial>
-      <origin xyz="0.062965 -0.000323 0.000692" />
-      <mass value="0.11904336"/>
-      <inertia ixx="0.097950272"  ixy="0.0012119368"  ixz="-0.00021223016" iyx="0.00122119368" iyy="0.032848287" iyz="-0.0019474021" izx="-0.00021223016" izy="-0.0019474021" izz="0.11493509" />
-    </inertial>
-    <thigh2_r_collision_geom_macro />
-    <thigh2_r_visual_geom_macro />
-  </link>
-  <link name="MP_TIBIA_R" >
-    <inertial>
-      <origin xyz="0.053955 0.006548 -0.000592" />
-      <mass value="0.070309794"/>
-      <inertia ixx="0.093369608"  ixy="-0.00093567395"  ixz="-0.00023992085" iyx="-0.00093567395" iyy="0.046295534" iyz="-0.012858493" izx="-0.00023992085" izy="-0.012858493" izz="0.11351516" />
-    </inertial>
-    <tibia_r_collision_geom_macro />
-    <tibia_r_visual_geom_macro />
-  </link>
-  <link name="MP_ANKLE1_R" >
-    <inertial>
-      <origin xyz="-0.000214 -0.018536 -0.013873" />
-      <mass value="0.16710792"/>
-      <inertia ixx="0.12079175"  ixy="-0.00079781067"  ixz="-0.00039322246" iyx="-0.00079781067" iyy="0.10885465" iyz="0.0070770117" izx="-0.00039322246" izy="0.0070770117" izz="0.041871103" />
-    </inertial>
-    <ankle1_r_collision_geom_macro />
-    <ankle1_r_visual_geom_macro />
-  </link>
-  <link name="MP_ANKLE2_R" >
-    <inertial>
-      <origin xyz="0.025995 -0.009506 -0.000503" />
-      <mass value="0.0794462"/>
-      <inertia ixx="0.12079175"  ixy="-0.00079781067"  ixz="-0.00039322246" iyx="-0.00079781067" iyy="0.10885465" iyz="0.0070770117" izx="-0.00039322246" izy="0.0070770117" izz="0.041871103" />
-    </inertial>
-    <ankle2_r_collision_geom_macro />
-    <ankle2_r_visual_geom_macro />
-  </link>
-  <joint name="j_pelvis_l" type="revolute">
-    <parent link="MP_BODY"/>
-    <child link="MP_PELVIS_L"/>
-    <origin xyz="-0.005 0.037 -0.09355" rpy="0 3.14159 -1.5707963" />
-    <axis xyz="0 0 1" />
-    <limit effort="2.8" velocity="5.6548668" lower="-2.6179939" upper="2.6179939" />
-  </joint>
-  <joint name="j_thigh1_l" type="revolute">
-    <parent link="MP_PELVIS_L"/>
-    <child link="MP_THIGH1_L"/>
-    <origin xyz="0 0 0.028652" rpy="1.5707963 0 0" />
-    <axis xyz="0 0 1" />
-    <limit effort="2.8" velocity="5.6548668" lower="-2.6179939" upper="2.6179939" />
-  </joint>
-  <joint name="j_thigh2_l" type="revolute">
-    <parent link="MP_THIGH1_L"/>
-    <child link="MP_THIGH2_L"/>
-    <origin xyz="0 0 0" rpy="1.5707963 0 -1.5707963" />
-    <axis xyz="0 0 1" />
-    <limit effort="2.8" velocity="5.6548668" lower="-2.6179939" upper="2.6179939" />
-  </joint>
-  <joint name="j_tibia_l" type="revolute">
-    <parent link="MP_THIGH2_L"/>
-    <child link="MP_TIBIA_L"/>
-    <origin xyz="-0.093 0 0" rpy="0 0 0" />
-    <axis xyz="0 0 1" />
-    <limit effort="2.8" velocity="5.6548668" lower="-2.6179939" upper="2.6179939" />
-  </joint>
-  <joint name="j_ankle1_l" type="revolute">
-    <parent link="MP_TIBIA_L"/>
-    <child link="MP_ANKLE1_L"/>
-    <origin xyz="-0.093 0 0" rpy="3.14159 0 0" />
-    <axis xyz="0 0 1" />
-    <limit effort="2.8" velocity="5.6548668" lower="-2.6179939" upper="2.6179939" />
-  </joint>
-  <joint name="j_ankle2_l" type="revolute">
-    <parent link="MP_ANKLE1_L"/>
-    <child link="MP_ANKLE2_L"/>
-    <origin xyz="0 0 0" rpy="-1.5707963 0 0" />
-    <axis xyz="0 0 1" />
-    <limit effort="2.8" velocity="5.6548668" lower="-2.6179939" upper="2.6179939" />
-  </joint>
-  <joint name="j_pelvis_r" type="revolute">
-    <parent link="MP_BODY"/>
-    <child link="MP_PELVIS_R"/>
-    <origin xyz="-0.005 -0.037 -0.09355" rpy="0 3.14159 1.5707963" />
-    <axis xyz="0 0 1" />
-    <limit effort="2.8" velocity="5.6548668" lower="-2.6179939" upper="2.6179939" />
-  </joint>
-  <joint name="j_thigh1_r" type="revolute">
-    <parent link="MP_PELVIS_R"/>
-    <child link="MP_THIGH1_R"/>
-    <origin xyz="0 0 0.028652" rpy="-1.5707963 0 0" />
-    <axis xyz="0 0 1" />
-    <limit effort="2.8" velocity="5.6548668" lower="-2.6179939" upper="2.6179939" />
-  </joint>
-  <joint name="j_thigh2_r" type="revolute">
-    <parent link="MP_THIGH1_R"/>
-    <child link="MP_THIGH2_R"/>
-    <origin xyz="0 0 0" rpy="1.5707963 0 -1.5707963" />
-    <axis xyz="0 0 1" />
-    <limit effort="2.8" velocity="5.6548668" lower="-2.6179939" upper="2.6179939" />
-  </joint>
-  <joint name="j_tibia_r" type="revolute">
-    <parent link="MP_THIGH2_R"/>
-    <child link="MP_TIBIA_R"/>
-    <origin xyz="0.093 0 0" rpy="0 0 0" />
-    <axis xyz="0 0 1" />
-    <limit effort="2.8" velocity="5.6548668" lower="-2.6179939" upper="2.6179939" />
-  </joint>
-  <joint name="j_ankle1_r" type="revolute">
-    <parent link="MP_TIBIA_R"/>
-    <child link="MP_ANKLE1_R"/>
-    <origin xyz="0.093 0 0" rpy="3.14159 0 0" />
-    <axis xyz="0 0 1" />
-    <limit effort="2.8" velocity="5.6548668" lower="-2.6179939" upper="2.6179939" />
-  </joint>
-  <joint name="j_ankle2_r" type="revolute">
-    <parent link="MP_ANKLE1_R"/>
-    <child link="MP_ANKLE2_R"/>
-    <origin xyz="0 0 0" rpy="-1.5707963 0 0" />
-    <axis xyz="0 0 1" />
-    <limit effort="2.8" velocity="5.6548668" lower="-2.6179939" upper="2.6179939" />
-  </joint>
-  <joint_transmission_macro joint_name="j_pelvis_l"/>
-  <joint_transmission_macro joint_name="j_thigh1_l"/>
-  <joint_transmission_macro joint_name="j_thigh2_l"/>
-  <joint_transmission_macro joint_name="j_tibia_l"/>
-  <joint_transmission_macro joint_name="j_ankle1_l"/>
-  <joint_transmission_macro joint_name="j_ankle2_l"/>
-  <joint_transmission_macro joint_name="j_pelvis_r"/>
-  <joint_transmission_macro joint_name="j_thigh1_r"/>
-  <joint_transmission_macro joint_name="j_thigh2_r"/>
-  <joint_transmission_macro joint_name="j_tibia_r"/>
-  <joint_transmission_macro joint_name="j_ankle1_r"/>
-  <joint_transmission_macro joint_name="j_ankle2_r"/>
-<gazebo reference="MP_ANKLE2_L">
-    <material>Gazebo/White</material>
-    <mu1>9000</mu1>
-    <mu2>9000</mu2>
-    <kp>1000000.0</kp>
-    <kd>10.0</kd>
-    <minDepth>0.000001</minDepth>
-    <maxContacts>100</maxContacts>
-  </gazebo>
-<gazebo reference="MP_ANKLE2_R">
-    <material>Gazebo/White</material>
-    <mu1>9000</mu1>
-    <mu2>9000</mu2>
-    <kp>1000000.0</kp>
-    <kd>10.0</kd>
-    <minDepth>0.000001</minDepth>
-    <maxContacts>100</maxContacts>
-  </gazebo>
+      </inertial>
+      <pelvis_l_collision_geom_macro />
+      <pelvis_l_visual_geom_macro />
+    </link>
+    <link name="MP_THIGH1_L" >
+      <inertial>
+        <origin xyz="0.000079 0.018242 0.013873" />
+        <mass value="0.11904336"/>
+        <inertia ixx="0.097950272"  ixy="0.0012119368"  ixz="-0.00021223016" iyx="0.00122119368" iyy="0.032848287" iyz="-0.0019474021" izx="-0.00021223016" izy="-0.0019474021" izz="0.11493509" />
+      </inertial>
+      <thigh1_l_collision_geom_macro />
+      <thigh1_l_visual_geom_macro />
+    </link>
+    <link name="MP_THIGH2_L" >
+      <inertial>
+        <origin xyz="-0.062965 -0.000323 0.000692" />
+        <mass value="0.11904336"/>
+        <inertia ixx="0.097950272"  ixy="0.0012119368"  ixz="-0.00021223016" iyx="0.00122119368" iyy="0.032848287" iyz="-0.0019474021" izx="-0.00021223016" izy="-0.0019474021" izz="0.11493509" />
+      </inertial>
+      <thigh2_l_collision_geom_macro />
+      <thigh2_l_visual_geom_macro />
+    </link>
+    <link name="MP_TIBIA_L" >
+      <inertial>
+        <origin xyz="-0.053955 0.006548 -0.000592" />
+        <mass value="0.070309794"/>
+        <inertia ixx="0.093369608"  ixy="-0.00093567395"  ixz="-0.00023992085" iyx="-0.00093567395" iyy="0.046295534" iyz="-0.012858493" izx="-0.00023992085" izy="-0.012858493" izz="0.11351516" />
+      </inertial>
+      <tibia_l_collision_geom_macro />
+      <tibia_l_visual_geom_macro />
+    </link>
+    <link name="MP_ANKLE1_L" >
+      <inertial>
+        <origin xyz="-0.000214 -0.018536 0.013873" />
+        <mass value="0.16710792"/>
+        <inertia ixx="0.12079175"  ixy="-0.00079781067"  ixz="-0.00039322246" iyx="-0.00079781067" iyy="0.10885465" iyz="0.0070770117" izx="-0.00039322246" izy="0.0070770117" izz="0.041871103" />
+      </inertial>
+      <ankle1_l_collision_geom_macro />
+      <ankle1_l_visual_geom_macro />
+    </link>
+    <link name="MP_ANKLE2_L" >
+      <inertial>
+        <origin xyz="-0.025995 -0.009506 -0.000503" />
+        <mass value="0.0794462"/>
+        <inertia ixx="0.12079175"  ixy="-0.00079781067"  ixz="-0.00039322246" iyx="-0.00079781067" iyy="0.10885465" iyz="0.0070770117" izx="-0.00039322246" izy="0.0070770117" izz="0.041871103" />
+      </inertial>
+      <ankle2_l_collision_geom_macro />
+      <ankle2_l_visual_geom_macro />
+    </link>
+    <link name="MP_PELVIS_R" >
+      <inertial>
+        <origin xyz="0.000000 0.000480 0.018437" />
+        <mass value="0.197"/>
+        <inertia ixx="0.12259691"  ixy="0.00071127469"  ixz="0.00081143913" iyx="0.00071127469" iyy="0.11066637" iyz="-0.0071635476" izx="0.00081143913" izy="-0.0071635476" izz="0.041877668" />
+      </inertial>
+      <pelvis_r_collision_geom_macro />
+      <pelvis_r_visual_geom_macro />
+    </link>
+    <link name="MP_THIGH1_R" >
+      <inertial>
+        <origin xyz="0.000079 -0.018242 0.0138735" />
+        <mass value="0.11904336"/>
+        <inertia ixx="0.097950272"  ixy="0.0012119368"  ixz="-0.00021223016" iyx="0.00122119368" iyy="0.032848287" iyz="-0.0019474021" izx="-0.00021223016" izy="-0.0019474021" izz="0.11493509" />
+      </inertial>
+      <thigh1_r_collision_geom_macro />
+      <thigh1_r_visual_geom_macro />
+    </link>
+    <link name="MP_THIGH2_R" >
+      <inertial>
+        <origin xyz="0.062965 -0.000323 0.000692" />
+        <mass value="0.11904336"/>
+        <inertia ixx="0.097950272"  ixy="0.0012119368"  ixz="-0.00021223016" iyx="0.00122119368" iyy="0.032848287" iyz="-0.0019474021" izx="-0.00021223016" izy="-0.0019474021" izz="0.11493509" />
+      </inertial>
+      <thigh2_r_collision_geom_macro />
+      <thigh2_r_visual_geom_macro />
+    </link>
+    <link name="MP_TIBIA_R" >
+      <inertial>
+        <origin xyz="0.053955 0.006548 -0.000592" />
+        <mass value="0.070309794"/>
+        <inertia ixx="0.093369608"  ixy="-0.00093567395"  ixz="-0.00023992085" iyx="-0.00093567395" iyy="0.046295534" iyz="-0.012858493" izx="-0.00023992085" izy="-0.012858493" izz="0.11351516" />
+      </inertial>
+      <tibia_r_collision_geom_macro />
+      <tibia_r_visual_geom_macro />
+    </link>
+    <link name="MP_ANKLE1_R" >
+      <inertial>
+        <origin xyz="-0.000214 -0.018536 -0.013873" />
+        <mass value="0.16710792"/>
+        <inertia ixx="0.12079175"  ixy="-0.00079781067"  ixz="-0.00039322246" iyx="-0.00079781067" iyy="0.10885465" iyz="0.0070770117" izx="-0.00039322246" izy="0.0070770117" izz="0.041871103" />
+      </inertial>
+      <ankle1_r_collision_geom_macro />
+      <ankle1_r_visual_geom_macro />
+    </link>
+    <link name="MP_ANKLE2_R" >
+      <inertial>
+        <origin xyz="0.025995 -0.009506 -0.000503" />
+        <mass value="0.0794462"/>
+        <inertia ixx="0.12079175"  ixy="-0.00079781067"  ixz="-0.00039322246" iyx="-0.00079781067" iyy="0.10885465" iyz="0.0070770117" izx="-0.00039322246" izy="0.0070770117" izz="0.041871103" />
+      </inertial>
+      <ankle2_r_collision_geom_macro />
+      <ankle2_r_visual_geom_macro />
+    </link>
+    <joint name="j_pelvis_l" type="revolute">
+      <parent link="MP_BODY"/>
+      <child link="MP_PELVIS_L"/>
+      <origin xyz="-0.005 0.037 -0.09355" rpy="0 3.14159 -1.5707963" />
+      <axis xyz="0 0 1" />
+      <limit effort="2.8" velocity="5.6548668" lower="-2.6179939" upper="2.6179939" />
+    </joint>
+    <joint name="j_thigh1_l" type="revolute">
+      <parent link="MP_PELVIS_L"/>
+      <child link="MP_THIGH1_L"/>
+      <origin xyz="0 0 0.028652" rpy="1.5707963 0 0" />
+      <axis xyz="0 0 1" />
+      <limit effort="2.8" velocity="5.6548668" lower="-2.6179939" upper="2.6179939" />
+    </joint>
+    <joint name="j_thigh2_l" type="revolute">
+      <parent link="MP_THIGH1_L"/>
+      <child link="MP_THIGH2_L"/>
+      <origin xyz="0 0 0" rpy="1.5707963 0 -1.5707963" />
+      <axis xyz="0 0 1" />
+      <limit effort="2.8" velocity="5.6548668" lower="-2.6179939" upper="2.6179939" />
+    </joint>
+    <joint name="j_tibia_l" type="revolute">
+      <parent link="MP_THIGH2_L"/>
+      <child link="MP_TIBIA_L"/>
+      <origin xyz="-0.093 0 0" rpy="0 0 0" />
+      <axis xyz="0 0 1" />
+      <limit effort="2.8" velocity="5.6548668" lower="-2.6179939" upper="2.6179939" />
+    </joint>
+    <joint name="j_ankle1_l" type="revolute">
+      <parent link="MP_TIBIA_L"/>
+      <child link="MP_ANKLE1_L"/>
+      <origin xyz="-0.093 0 0" rpy="3.14159 0 0" />
+      <axis xyz="0 0 1" />
+      <limit effort="2.8" velocity="5.6548668" lower="-2.6179939" upper="2.6179939" />
+    </joint>
+    <joint name="j_ankle2_l" type="revolute">
+      <parent link="MP_ANKLE1_L"/>
+      <child link="MP_ANKLE2_L"/>
+      <origin xyz="0 0 0" rpy="-1.5707963 0 0" />
+      <axis xyz="0 0 1" />
+      <limit effort="2.8" velocity="5.6548668" lower="-2.6179939" upper="2.6179939" />
+    </joint>
+    <gazebo reference="j_ankle2_l">
+      <provideFeedback>true</provideFeedback>
+    </gazebo>
+    <joint name="j_pelvis_r" type="revolute">
+      <parent link="MP_BODY"/>
+      <child link="MP_PELVIS_R"/>
+      <origin xyz="-0.005 -0.037 -0.09355" rpy="0 3.14159 1.5707963" />
+      <axis xyz="0 0 1" />
+      <limit effort="2.8" velocity="5.6548668" lower="-2.6179939" upper="2.6179939" />
+    </joint>
+    <joint name="j_thigh1_r" type="revolute">
+      <parent link="MP_PELVIS_R"/>
+      <child link="MP_THIGH1_R"/>
+      <origin xyz="0 0 0.028652" rpy="-1.5707963 0 0" />
+      <axis xyz="0 0 1" />
+      <limit effort="2.8" velocity="5.6548668" lower="-2.6179939" upper="2.6179939" />
+    </joint>
+    <joint name="j_thigh2_r" type="revolute">
+      <parent link="MP_THIGH1_R"/>
+      <child link="MP_THIGH2_R"/>
+      <origin xyz="0 0 0" rpy="1.5707963 0 -1.5707963" />
+      <axis xyz="0 0 1" />
+      <limit effort="2.8" velocity="5.6548668" lower="-2.6179939" upper="2.6179939" />
+    </joint>
+    <joint name="j_tibia_r" type="revolute">
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